File: Hardware/RS232/PCB.brd (EAGLE design)
At the start: 32.4 x 29.2 mm, 20 parts, among them U1 SP3232XTSSOP

Commit message: RS232 Files
Parts:
- added RX, TX: JUMPER-SMT_2_NC_TRACE_SILK, SparkFun-Jumpers:SMT-JUMPER_2_NC_TRACE_SILK
- TTL: value PINHD-1X4/90 -> B6B-PH-K-S(LF)(SN); device Connector:1X04/90 -> B6B-PH-K-S_LF__SN_:JST_B6B-PH-K-S(LF)(SN)
- moved TTL 8.28 mm to (23.3, 26.0), turned to 180 degrees
- moved R1 3.40 mm to (27.5, 21.1), turned to 0 degrees
- moved R2 3.40 mm to (20.5, 21.1), turned to 180 degrees
- moved C1 1.27 mm to (28.7, 15.2)
- moved C4 1.27 mm to (21.7, 13.6)
- moved C2 1.27 mm to (28.7, 18.3)
- moved C3 1.27 mm to (30.3, 17.3)
- moved RXD 1.27 mm to (25.2, 21.1)
- moved TXD 1.27 mm to (22.7, 21.1)
- moved U1 1.27 mm to (24.0, 17.6)
- moved JP1 0.25 mm to (15.0, 18.3)
Connections:
- net R1_IN: now also TX.2
- net R1_OUT: now also TTL.3; no longer TTL.2
- net RS232_RXD: now also RX.1
- net RS232_TXD: now also TX.1
- net T1_IN: now also TTL.6; no longer TTL.3
- net T1_OUT: now also RX.2
Routing:
- net 3V3: track 37.2 -> 47.6 mm
- net RS232_RXD: track 7.92 -> 12.0 mm
- net R1_IN: track 8.18 -> 11.5 mm
- net RS232_TXD: track 8.43 -> 11.3 mm
- net T1_OUT: track 7.95 -> 10.1 mm
- net R1_OUT: track 15.7 -> 14.3 mm, vias 0 -> 1
Other:
- board text added: "RS232-TTL strenuous.dev"
- board text added: "TX GN RX 3V"
- board text removed: "3V R T G"
- board text removed: "RS232-TTL ripper121.com"
